Commit message: Update tool mesh and URDF

File: urdf/mr3_mini.urdf (robot description, URDF)
Before this commit: robot mr3_mini, 23 links, 22 joints
Joints:
- joint flange_to_tool_base: origin xyz=0 0 0 rpy=0 0 0 -> xyz=0 0 -0.026 rpy=0 0 0
- joint tool_base_to_x_axis: origin xyz=0.0085 0 -0.026 rpy=0 0 0 -> xyz=0.0085 0 0 rpy=0 0 0
- joint tool_base_to_y_axis: origin xyz=0 0.0085 -0.026 rpy=0 0 0 -> xyz=0 0.0085 0 rpy=0 0 0
- joint tool_base_to_z_axis: origin xyz=0 0 -0.0345 rpy=0 0 0 -> xyz=0 0 -0.0085 rpy=0 0 0
